File: rgb_no_bootloader.kicad_sch (KiCad schematic)
At the start: 9 parts, among them J1 USB-C fingers, J2 FFC programming interface, U1 ATtiny84A-CC

Commit message: Finished routing Demo 2, added Demo 4, updated readme with newer findings
Parts:
- C1: footprint Capacitor_SMD:C_0402_1005Metric -> Capacitor_SMD:C_0201_0603Metric
Changed lines of the file:
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@@
     (property "Reference" "C1" (id 0) (at 106.68 28.5242 90))
     (property "Value" "0.1u" (id 1) (at 106.68 30.8356 90))
-    (property "Footprint" "Capacitor_SMD:C_0402_1005Metric" (id 2) (at 102.87 35.8902 0)
+    (property "Footprint" "Capacitor_SMD:C_0201_0603Metric" (id 2) (at 102.87 35.8902 0)
       (effects (font (size 1.27 1.27)) hide)
     )
