File: rgb_no_bootloader_r2.kicad_sch (KiCad schematic)
At the start: 9 parts, among them J10 FFC programming interface, J9 USB-C fingers, U4 ATtiny84A-CC

Commit message: Finished routing Demo 2, added Demo 4, updated readme with newer findings
Parts:
- C4: footprint Capacitor_SMD:C_0402_1005Metric -> Capacitor_SMD:C_0201_0603Metric
Changed lines of the file:
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@@
     (property "Reference" "C4" (id 0) (at 126.365 32.3342 90))
     (property "Value" "0.1u" (id 1) (at 126.365 34.6456 90))
-    (property "Footprint" "Capacitor_SMD:C_0402_1005Metric" (id 2) (at 122.555 39.7002 0)
+    (property "Footprint" "Capacitor_SMD:C_0201_0603Metric" (id 2) (at 122.555 39.7002 0)
       (effects (font (size 1.27 1.27)) hide)
     )
